File: esp32.kicad_sch (KiCad schematic)
At the start: 46 parts, among them J5 Conn_01x05, SW2 BOOT, U6 ESP32-S3R8, U7 W25Q128JVSIQ, Y1 40MHz

Commit message: 1st test batch
Parts:
- TP6, TP7: now not fitted
