File: esp32.kicad_sch (KiCad schematic)
At the start: 46 parts, among them J5 Conn_01x05, SW2 BOOT, U6 ESP32-S3R8, U7 W25Q128JVSIQ, Y1 40MHz

Commit message: Production update
Parts:
- SW2: Purchase-URL (none) -> https://www.lcsc.com/product-detail/C221897.html?s_z=n_PTS8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
- Y1: Purchase-URL (none) -> https://www.lcsc.com/product-detail/C424431.html?s_z=n_TAXM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
Changed lines of the file:
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@@
+			)
+		)
+		(property "Purchase-URL" "https://www.lcsc.com/product-detail/C424431.html?s_z=n_TAXM40M4ZCBCDT2T"
+			(at 64.77 85.09 90)
+			(effects
+				(font
+					(size 1.27 1.27)
+				)
+				(hide yes)
 			)
 		)
@@
 			(at 91.44 177.8 90)
 			(effects
+				(font
+					(size 1.27 1.27)
+				)
+				(hide yes)
+			)
+		)
+		(property "Purchase-URL" "https://www.lcsc.com/product-detail/C221897.html?s_z=n_PTS810SJS250SMTRLFS"
+			(at 91.44 177.8 90)
+			(effects
