File: audio.kicad_sch (KiCad schematic)
At the start: 51 parts, among them J2 1775443-2, U13 TLV320AIC3204IRHBR, U14 TPA6211A1DGNR

Commit message: 1st test batch
Parts:
- FB7, FB8: footprint Inductor_SMD:L_0603_1608Metric -> Onju:BLM18PG121SN1D

Commit message: Production update
Parts:
- C76, C89, C91: Purchase-URL (none) -> https://www.lcsc.com/product-detail/C19702.html?s_z=n_CL10A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
Changed lines of the file:
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@@
 			)
 		)
+		(property "Purchase-URL" "https://www.lcsc.com/product-detail/C19702.html?s_z=n_CL10A106KP8NNNC"
+			(at 161.29 74.93 0)
+			(effects
+				(font
+					(size 1.27 1.27)
+				)
+				(hide yes)
+			)
+		)
 		(pin "2"
 		)
@@
 			)
 		)
+		(property "Purchase-URL" "https://www.lcsc.com/product-detail/C19702.html?s_z=n_CL10A106KP8NNNC"
+			(at 48.26 163.83 0)
+			(effects
+				(font
+					(size 1.27 1.27)
+				)
+				(hide yes)
+			)
+		)
 		(pin "1"
 		)
@@
 			(at 166.37 162.56 0)
 			(effects
+				(font
+					(size 1.27 1.27)
+				)
+				(hide yes)
+			)
+		)
+		(property "Purchase-URL" "https://www.lcsc.com/product-detail/C19702.html?s_z=n_CL10A106KP8NNNC"
+			(at 166.37 162.56 0)
+			(effects
